File: Adapter-IOX-test_array.brd (EAGLE design)
At the start: 110.5 x 114.3 mm, 317 parts, among them Q0X11 P-FET, Q0X12 P-FET, Q0X13 P-FET, Q0X21 P-FET, Q0X22 P-FET, Q0X23 P-FET, Q10X11 P-FET, Q10X12 P-FET, Q10X13 P-FET, Q10X21 P-FET, Q10X22 P-FET, Q10X23 P-FET, Q11X11 P-FET, Q11X12 P-FET, Q11X13 P-FET, Q11X21 P-FET, Q11X22 P-FET, Q11X23 P-FET, Q12X11 P-FET, Q12X12 P-FET, Q12X13 P-FET, Q12X21 P-FET, Q12X22 P-FET, Q12X23 P-FET, Q13X11 P-FET, Q13X12 P-FET, Q13X13 P-FET, Q13X21 P-FET, Q13X22 P-FET, Q13X23 P-FET, Q14X11 P-FET, Q14X12 P-FET, Q14X13 P-FET, Q14X21 P-FET, Q14X22 P-FET, Q14X23 P-FET, Q15X11 P-FET, Q15X12 P-FET, Q15X13 P-FET, Q15X21 P-FET, Q15X22 P-FET, Q15X23 P-FET, Q1X11 P-FET, Q1X12 P-FET, Q1X13 P-FET, Q1X21 P-FET, Q1X22 P-FET, Q1X23 P-FET, Q2X11 P-FET, Q2X12 P-FET, Q2X13 P-FET, Q2X21 P-FET, Q2X22 P-FET, Q2X23 P-FET, Q3X11 P-FET, Q3X12 P-FET, Q3X13 P-FET, Q3X21 P-FET, Q3X22 P-FET, Q3X23 P-FET, Q4X11 P-FET, Q4X12 P-FET, Q4X13 P-FET, Q4X21 P-FET, Q4X22 P-FET, Q4X23 P-FET, Q5X11 P-FET, Q5X12 P-FET, Q5X13 P-FET, Q5X21 P-FET, Q5X22 P-FET, Q5X23 P-FET, Q6X11 P-FET, Q6X12 P-FET, Q6X13 P-FET, Q6X21 P-FET, Q6X22 P-FET, Q6X23 P-FET, Q7X11 P-FET, Q7X12 P-FET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

Commit message: added values for connectors
Parts:
- CON1X11, CON1X12, CON1X13, CON1X21, CON1X22, CON1X23, CON2X11, CON2X12, CON2X13, CON2X21, CON2X22, CON2X23, J1X11, J1X12, J1X13, J1X21, J1X22, J1X23, J2X11, J2X12, J2X13, J2X21, J2X22, J2X23: value (none) -> 0.100
- FID1, FID3: value (none) -> FID
- R22X1: value (none) -> 10x10
Changed lines of the file:
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@@
 </autorouter>
 <elements>
-<element name="CON1X11" library="SPCoast" package="1X02_LOCK" value="" x="2.413" y="20.0152"/>
-<element name="CON2X11" library="SPCoast" package="1X02_LOCK" value="" x="2.413" y="17.399"/>
-<element name="J1X11" library="SPCoast" package="1X08_LOCK" value="" x="42.5704" y="33.7312" rot="R180"/>
-<element name="J2X11" library="SPCoast" package="1X08_LOCK" value="" x="22.2504" y="33.7312" rot="R180"/>
+<element name="CON1X11" library="SPCoast" package="1X02_LOCK" value="0.100" x="2.413" y="20.0152"/>
+<element name="CON2X11" library="SPCoast" package="1X02_LOCK" value="0.100" x="2.413" y="17.399"/>
+<element name="J1X11" library="SPCoast" package="1X08_LOCK" value="0.100" x="42.5704" y="33.7312" rot="R180"/>
+<element name="J2X11" library="SPCoast" package="1X08_LOCK" value="0.100" x="22.2504" y="33.7312" rot="R180"/>
 <element name="LED1X11" library="SPCoast" package="0603-LED" value="Y" x="41.656" y="10.2108" rot="R90"/>
 <element name="LED2X11" library="SPCoast" package="0603-LED" value="Y" x="39.116" y="10.2108" rot="R90"/>
@@
 <element name="R21X11" library="SPCoast" package="0805-RES" value="2K0" x="3.556" y="14.0208" rot="R90"/>
 <element name="R22X11" library="SPCoast" package="0805-RES" value="2K0" x="11.176" y="14.0208" rot="R90"/>
-<element name="CON1X12" library="SPCoast" package="1X02_LOCK" value="" x="2.413" y="47.9552"/>
-<element name="CON2X12" library="SPCoast" package="1X02_LOCK" value="" x="2.413" y="45.339"/>
-<element name="J1X12" library="SPCoast" package="1X08_LOCK" value="" x="42.5704" y="61.6712" rot="R180"/>
-<element name="J2X12" library="SPCoast" package="1X08_LOCK" value="" x="22.2504" y="61.6712" rot="R180"/>
+<element name="CON1X12" library="SPCoast" package="1X02_LOCK" value="0.100" x="2.413" y="47.9552"/>
+<element name="CON2X12" library="SPCoast" package="1X02_LOCK" value="0.100" x="2.413" y="45.339"/>
+<element name="J1X12" library="SPCoast" package="1X08_LOCK" value="0.100" x="42.5704" y="61.6712" rot="R180"/>
+<element name="J2X12" library="SPCoast" package="1X08_LOCK" value="0.100" x="22.2504" y="61.6712" rot="R180"/>
 <element name="LED1X12" library="SPCoast" package="0603-LED" value="Y" x="41.656" y="38.1508" rot="R90"/>
 <element name="LED2X12" library="SPCoast" package="0603-LED" value="Y" x="39.116" y="38.1508" rot="R90"/>
@@
 <element name="R21X12" library="SPCoast" package="0805-RES" value="2K0" x="3.556" y="41.9608" rot="R90"/>
 <element name="R22X12" library="SPCoast" package="0805-RES" value="2K0" x="11.176" y="41.9608" rot="R90"/>
-<element name="CON1X13" library="SPCoast" package="1X02_LOCK" value="" x="2.413" y="75.8952"/>
-<element name="CON2X13" library="SPCoast" package="1X02_LOCK" value="" x="2.413" y="73.279"/>
-<element name="J1X13" library="SPCoast" package="1X08_LOCK" value="" x="42.5704" y="89.6112" rot="R180"/>
-<element name="J2X13" library="SPCoast" package="1X08_LOCK" value="" x="22.2504" y="89.6112" rot="R180"/>
+<element name="CON1X13" library="SPCoast" package="1X02_LOCK" value="0.100" x="2.413" y="75.8952"/>
+<element name="CON2X13" library="SPCoast" package="1X02_LOCK" value="0.100" x="2.413" y="73.279"/>
+<element name="J1X13" library="SPCoast" package="1X08_LOCK" value="0.100" x="42.5704" y="89.6112" rot="R180"/>
+<element name="J2X13" library="SPCoast" package="1X08_LOCK" value="0.100" x="22.2504" y="89.6112" rot="R180"/>
 <element name="LED1X13" library="SPCoast" package="0603-LED" value="Y" x="41.656" y="66.0908" rot="R90"/>
 <element name="LED2X13" library="SPCoast" package="0603-LED" value="Y" x="39.116" y="66.0908" rot="R90"/>
@@
 <element name="R21X13" library="SPCoast" package="0805-RES" value="2K0" x="3.556" y="69.9008" rot="R90"/>
 <element name="R22X13" library="SPCoast" package="0805-RES" value="2K0" x="11.176" y="69.9008" rot="R90"/>
-<element name="CON1X21" library="SPCoast" package="1X02_LOCK" value="" x="46.863" y="20.0152"/>
-<element name="CON2X21" library="SPCoast" package="1X02_LOCK" value="" x="46.863" y="17.399"/>
-<element name="J1X21" library="SPCoast" package="1X08_LOCK" value="" x="87.0204" y="33.7312" rot="R180"/>
-<element name="J2X21" library="SPCoast" package="1X08_LOCK" value="" x="66.7004" y="33.7312" rot="R180"/>
+<element name="CON1X21" library="SPCoast" package="1X02_LOCK" value="0.100" x="46.863" y="20.0152"/>
+<element name="CON2X21" library="SPCoast" package="1X02_LOCK" value="0.100" x="46.863" y="17.399"/>
+<element name="J1X21" library="SPCoast" package="1X08_LOCK" value="0.100" x="87.0204" y="33.7312" rot="R180"/>
+<element name="J2X21" library="SPCoast" package="1X08_LOCK" value="0.100" x="66.7004" y="33.7312" rot="R180"/>
 <element name="LED1X21" library="SPCoast" package="0603-LED" value="Y" x="86.106" y="10.2108" rot="R90"/>
 <element name="LED2X21" library="SPCoast" package="0603-LED" value="Y" x="83.566" y="10.2108" rot="R90"/>
@@
 <element name="R21X21" library="SPCoast" package="0805-RES" value="2K0" x="48.006" y="14.0208" rot="R90"/>
 <element name="R22X21" library="SPCoast" package="0805-RES" value="2K0" x="55.626" y="14.0208" rot="R90"/>
-<element name="CON1X22" library="SPCoast" package="1X02_LOCK" value="" x="46.863" y="47.9552"/>
-<element name="CON2X22" library="SPCoast" package="1X02_LOCK" value="" x="46.863" y="45.339"/>
-<element name="J1X22" library="SPCoast" package="1X08_LOCK" value="" x="87.0204" y="61.6712" rot="R180"/>
-<element name="J2X22" library="SPCoast" package="1X08_LOCK" value="" x="66.7004" y="61.6712" rot="R180"/>
+<element name="CON1X22" library="SPCoast" package="1X02_LOCK" value="0.100" x="46.863" y="47.9552"/>
+<element name="CON2X22" library="SPCoast" package="1X02_LOCK" value="0.100" x="46.863" y="45.339"/>
+<element name="J1X22" library="SPCoast" package="1X08_LOCK" value="0.100" x="87.0204" y="61.6712" rot="R180"/>
+<element name="J2X22" library="SPCoast" package="1X08_LOCK" value="0.100" x="66.7004" y="61.6712" rot="R180"/>
 <element name="LED1X22" library="SPCoast" package="0603-LED" value="Y" x="86.106" y="38.1508" rot="R90"/>
 <element name="LED2X22" library="SPCoast" package="0603-LED" value="Y" x="83.566" y="38.1508" rot="R90"/>
@@
 <element name="R21X22" library="SPCoast" package="0805-RES" value="2K0" x="48.006" y="41.9608" rot="R90"/>
 <element name="R22X22" library="SPCoast" package="0805-RES" value="2K0" x="55.626" y="41.9608" rot="R90"/>
-<element name="CON1X23" library="SPCoast" package="1X02_LOCK" value="" x="46.863" y="75.8952"/>
-<element name="CON2X23" library="SPCoast" package="1X02_LOCK" value="" x="46.863" y="73.279"/>
-<element name="J1X23" library="SPCoast" package="1X08_LOCK" value="" x="87.0204" y="89.6112" rot="R180"/>
-<element name="J2X23" library="SPCoast" package="1X08_LOCK" value="" x="66.7004" y="89.6112" rot="R180"/>
+<element name="CON1X23" library="SPCoast" package="1X02_LOCK" value="0.100" x="46.863" y="75.8952"/>
+<element name="CON2X23" library="SPCoast" package="1X02_LOCK" value="0.100" x="46.863" y="73.279"/>
+<element name="J1X23" library="SPCoast" package="1X08_LOCK" value="0.100" x="87.0204" y="89.6112" rot="R180"/>
+<element name="J2X23" library="SPCoast" package="1X08_LOCK" value="0.100" x="66.7004" y="89.6112" rot="R180"/>
 <element name="LED1X23" library="SPCoast" package="0603-LED" value="Y" x="86.106" y="66.0908" rot="R90"/>
 <element name="LED2X23" library="SPCoast" package="0603-LED" value="Y" x="83.566" y="66.0908" rot="R90"/>
@@
 <element name="R21X23" library="SPCoast" package="0805-RES" value="2K0" x="48.006" y="69.9008" rot="R90"/>
 <element name="R22X23" library="SPCoast" package="0805-RES" value="2K0" x="55.626" y="69.9008" rot="R90"/>
-<element name="R22X1" library="SPCoast" package="BOARD-10X10-TEMPLATE" value="" x="0" y="0"/>
-<element name="FID1" library="SPCoast" package="FIDUCIAL_1MM" value="" x="2.54" y="93.98"/>
-<element name="FID3" library="SPCoast" package="FIDUCIAL_1MM" value="" x="91.44" y="5.08"/>
+<element name="R22X1" library="SPCoast" package="BOARD-10X10-TEMPLATE" value="10x10" x="0" y="0"/>
+<element name="FID1" library="SPCoast" package="FIDUCIAL_1MM" value="FID" x="2.54" y="93.98"/>
+<element name="FID3" library="SPCoast" package="FIDUCIAL_1MM" value="FID" x="91.44" y="5.08"/>
 <element name="FID2" library="SPCoast" package="FIDUCIAL_1MM" value="" x="97.79" y="93.345"/>
 <element name="FID4" library="SPCoast" package="FIDUCIAL_1MM" value="" x="8.89" y="5.08"/>

Commit message: added values for connectors
Parts:
- FID2, FID4: value (none) -> FID
Changed lines of the file:
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@@
 <element name="FID1" library="SPCoast" package="FIDUCIAL_1MM" value="FID" x="2.54" y="93.98"/>
 <element name="FID3" library="SPCoast" package="FIDUCIAL_1MM" value="FID" x="91.44" y="5.08"/>
-<element name="FID2" library="SPCoast" package="FIDUCIAL_1MM" value="" x="97.79" y="93.345"/>
-<element name="FID4" library="SPCoast" package="FIDUCIAL_1MM" value="" x="8.89" y="5.08"/>
+<element name="FID2" library="SPCoast" package="FIDUCIAL_1MM" value="FID" x="97.79" y="93.345"/>
+<element name="FID4" library="SPCoast" package="FIDUCIAL_1MM" value="FID" x="8.89" y="5.08"/>
 </elements>
 <signals>

Commit message: normalized values
Parts:
- removed FID2, FID4: FID, SPCoast:FIDUCIAL_1MM
- FID-LR, FID-UL: value FID -> FIDUCIAL
- R22X1: value 10x10 -> BOARD
- renumbered FID1 to FID-UL, FID3 to FID-LR
Changed lines of the file:
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@@
 <element name="R21X23" library="SPCoast" package="0805-RES" value="2K0" x="48.006" y="69.9008" rot="R90"/>
 <element name="R22X23" library="SPCoast" package="0805-RES" value="2K0" x="55.626" y="69.9008" rot="R90"/>
-<element name="R22X1" library="SPCoast" package="BOARD-10X10-TEMPLATE" value="10x10" x="0" y="0"/>
-<element name="FID1" library="SPCoast" package="FIDUCIAL_1MM" value="FID" x="2.54" y="93.98"/>
-<element name="FID3" library="SPCoast" package="FIDUCIAL_1MM" value="FID" x="91.44" y="5.08"/>
-<element name="FID2" library="SPCoast" package="FIDUCIAL_1MM" value="FID" x="97.79" y="93.345"/>
-<element name="FID4" library="SPCoast" package="FIDUCIAL_1MM" value="FID" x="8.89" y="5.08"/>
+<element name="R22X1" library="SPCoast" package="BOARD-10X10-TEMPLATE" value="BOARD" x="0" y="0"/>
+<element name="FID-UL" library="SPCoast" package="FIDUCIAL_1MM" value="FIDUCIAL" x="2.54" y="93.98"/>
+<element name="FID-LR" library="SPCoast" package="FIDUCIAL_1MM" value="FIDUCIAL" x="91.44" y="5.08"/>
 </elements>
 <signals>
